Commit message: Migrate from Gazebo Fortress to Harmonic

File: parc_robot_description/urdf/gps.xacro (robot description, xacro)
@@ -19,20 +19,5 @@
         <update_rate>4.0</update_rate>
         <topic>gps/fix</topic>
-        <!-- <navsat> -->
-        <!--   <position_sensing> -->
-        <!--     <horizontal> -->
-        <!--       <noise type="gaussian"> -->
-        <!--         <mean>0.0</mean> -->
-        <!--         <stddev>0.001</stddev> -->
-        <!--       </noise> -->
-        <!--     </horizontal> -->
-        <!--     <vertical> -->
-        <!--       <noise type="gaussian"> -->
-        <!--         <mean>0.0</mean> -->
-        <!--         <stddev>0.001</stddev> -->
-        <!--       </noise> -->
-        <!--     </vertical> -->
-        <!--   </position_sensing> -->
-        <!-- </navsat> -->
+        <gz_frame_id>gps_link</gz_frame_id>
       </sensor>
     </gazebo>

File: parc_robot_description/urdf/parc_robot_gazebo.xacro (robot description, xacro)
@@ -1,7 +1,7 @@
 <?xml version="1.0"?>
 <robot xmlns:xacro="http://ros.org/wiki/xacro">
- <ros2_control name='IgnitionSystem' type='system'>
+  <ros2_control name="GazeboSimSystem" type="system">
     <hardware>
-      <plugin>ign_ros2_control/IgnitionSystem</plugin>
+      <plugin>gz_ros2_control/GazeboSimSystem</plugin>
     </hardware>
     <joint name='front_left_wheel'>
@@ -38,12 +38,9 @@
     </joint>
   </ros2_control>
- <gazebo>
-   <plugin filename="ign_ros2_control-system" name="ign_ros2_control::IgnitionROS2ControlPlugin">
-     <parameters>$(find parc_robot_bringup)/config/controllers.yaml</parameters>
-     <parameters>$(find parc_robot_bringup)/config/gazebo_ros2_ctl_use_sim.yaml</parameters>
-     <ros>
-         <remapping>/robot_base_controller/cmd_vel_unstamped:=/cmd_vel</remapping>
-     </ros>
-   </plugin>
- </gazebo>
+  <gazebo>
+    <plugin filename="libgz_ros2_control-system.so" name="gz_ros2_control::GazeboSimROS2ControlPlugin">
+       <parameters>$(find parc_robot_bringup)/config/controllers.yaml</parameters>
+       <parameters>$(find parc_robot_bringup)/config/gazebo_ros2_ctl_use_sim.yaml</parameters>
+    </plugin>
+  </gazebo>
 </robot>

File: parc_robot_description/urdf/side_cameras.xacro (robot description, xacro)
@@ -38,6 +38,5 @@
       <update_rate>30</update_rate>
       <topic>left_camera/image_raw</topic>
-      <gz_frame_id>left_camera_rgb_frame</gz_frame_id>
-      <!-- <gz_frame_id>camera_optical_frame</gz_frame_id> -->
+      <gz_frame_id>left_camera</gz_frame_id>
       <camera name="left_camera">
         <camera_info_topic>left_camera/camera_info</camera_info_topic>
@@ -104,6 +103,5 @@
       <update_rate>30</update_rate>
       <topic>right_camera/image_raw</topic>
-      <gz_frame_id>right_camera_rgb_frame</gz_frame_id>
-      <!-- <gz_frame_id>camera_optical_frame</gz_frame_id> -->
+      <gz_frame_id>right_camera</gz_frame_id>
       <camera name="right_camera">
         <camera_info_topic>right_camera/camera_info</camera_info_topic>

File: parc_robot_description/urdf/ydlidar.xacro (robot description, xacro)
@@ -25,17 +25,4 @@
       </collision>
     </link>
-    <!-- <link name="laser_frame">
-        <inertial>
-            <origin xyz="-0.00036659 0.00064155 -0.00027052" rpy="0 0 0" />
-            <mass value="0.25482" />
-            <inertia
-                ixx="8.9194E-05"
-                ixy="1.8116E-07"
-                ixz="3.6435E-08"
-                iyy="0.00018279"
-                iyz="2.423E-07"
-                izz="0.00011103" />
-        </inertial>
-    </link> -->
     <joint name="${name}_joint" type="fixed">
       <xacro:insert_block name="origin" />
@@ -50,5 +37,5 @@
         <update_rate>40</update_rate>
         <topic>scan</topic>
-        <gz_frame_id>base_scan</gz_frame_id>
+        <gz_frame_id>${name}_link</gz_frame_id>
         <lidar>
           <scan>
@@ -72,5 +59,4 @@
       </sensor>
     </gazebo>
-    <!-- Be mindful of gazebo reference and sensor names -->
   </xacro:macro>
 </robot>

File: parc_robot_description/urdf/zed2.xacro (robot description, xacro)
@@ -24,5 +24,5 @@
       </collision>
     </link>
-    <!-- Center Camera -->
+    <!-- Camera Center Joint -->
     <joint name="zed2_camera_center_joint" type="fixed">
       <xacro:insert_block name="origin" />
@@ -92,5 +92,8 @@
         <update_rate>30.0</update_rate>
         <visualize>false</visualize>
-        <camera name="zed2_center_camera">
+        <topic>zed2_camera_center/image_raw</topic>
+        <gz_frame_id>zed2_camera_center</gz_frame_id>
+        <camera name="zed2_camera_center">
+          <camera_info_topic>zed2_camera_center/camera_info</camera_info_topic>
           <horizontal_fov>1.9</horizontal_fov>
           <image>
@@ -117,15 +120,4 @@
           </distortion>
         </camera>
-        <plugin name="zed2_center_camera_controller" filename="libgazebo_ros_camera.so">
-          <cameraName>camera</cameraName>
-          <imageTopicName>image_raw</imageTopicName>
-          <cameraInfoTopicName>camera_info</cameraInfoTopicName>
-          <frameName>camera_optical_frame</frameName>
-          <distortionK1>-0.279817</distortionK1>
-          <distortionK2>0.060321</distortionK2>
-          <distortionK3>0.000487</distortionK3>
-          <distortionT1>0.000310</distortionT1>
-          <distortionT2>0.000000</distortionT2>
-        </plugin>
       </sensor>
     </gazebo>
@@ -163,5 +155,5 @@
           </distortion>
         </camera>
-        <plugin name="zed2_left_camera_controller" filename="libgazebo_ros_camera.so">
+        <!-- <plugin name="zed2_left_camera_controller" filename="libgazebo_ros_camera.so">
           <cameraName>zed2/left_raw</cameraName>
           <imageTopicName>image_raw_color</imageTopicName>
@@ -177,5 +169,5 @@
           <Cy>366.8340148925781</Cy>
           <hackBaseline>0.0</hackBaseline>
-        </plugin>
+        </plugin> -->
       </sensor>
       <sensor type="depth" name="zed2_leftd_camera">
@@ -202,9 +194,9 @@
           </noise>
         </camera>
-        <plugin name="zed2_leftd_camera_controller" filename="libgazebo_ros_camera.so">
-          <frame_name>zed2_left_camera_optical_frame</frame_name>
+        <!-- <plugin name="zed2_leftd_camera_controller" filename="libgazebo_ros_camera.so">
+          <frame_name>zed2_left_camera_optical_frame</frame_name> -->
           <!-- <min_depth>0.1</min_depth> -->
           <!-- <max_depth>100</max_depth> -->
-          <cameraName>zed2</cameraName>
+          <!-- <cameraName>zed2</cameraName>
           <imageTopicName>left/image_rect_color</imageTopicName>
           <cameraInfoTopicName>left/camera_info</cameraInfoTopicName>
@@ -219,5 +211,5 @@
           <Cy>372.25787353515625</Cy>
           <hackBaseline>0.0</hackBaseline>
-        </plugin>
+        </plugin> -->
       </sensor>
     </gazebo>
@@ -254,5 +246,5 @@
           </distortion>
         </camera>
-        <plugin name="zed2_right_camera_controller" filename="libgazebo_ros_camera.so">
+        <!-- <plugin name="zed2_right_camera_controller" filename="libgazebo_ros_camera.so">
           <cameraName>zed2/right_raw</cameraName>
           <imageTopicName>image_raw_color</imageTopicName>
@@ -268,5 +260,5 @@
           <Cy>371.39849853515625</Cy>
           <hackBaseline>0.12</hackBaseline>
-        </plugin>
+        </plugin> -->
       </sensor>
       <sensor type="camera" name="zed2_right_camera">
@@ -292,5 +284,5 @@
           </noise>
         </camera>
-        <plugin name="zed2_rightrect_camera_controller" filename="libgazebo_ros_camera.so">
+        <!-- <plugin name="zed2_rightrect_camera_controller" filename="libgazebo_ros_camera.so">
           <cameraName>zed2/right</cameraName>
           <imageTopicName>image_rect_color</imageTopicName>
@@ -301,23 +293,7 @@
           <Cy>372.25787353515625</Cy>
           <hackBaseline>0.12</hackBaseline>
-        </plugin>
+        </plugin> -->
       </sensor>
     </gazebo>
-    <!-- IMU -->
-    <!-- <gazebo reference="zed2_left_camera_frame">
-      <sensor type="imu" name="zed2_imu_sensor">
-        <update_rate>100</update_rate>
-        <plugin filename="libgazebo_ros_imu_sensor.so" name="imu_plugin">
-            <topicName>imu</topicName>
-            <bodyName>imu_link</bodyName>
-            <updateRateHZ>10.0</updateRateHZ>
-            <gaussianNoise>0.0</gaussianNoise>
-            <xyzOffset>0 0 0</xyzOffset>
-            <rpyOffset>0 0 0</rpyOffset>
-            <frame_name>imu_link</frame_name>
-            <initialOrientationAsReference>false</initialOrientationAsReference>
-        </plugin>
-      </sensor> -->
-    <!-- </gazebo> -->
   </xacro:macro>
 </robot>
