Commit message: Update world and config files

File: parc_robot_description/urdf/parc_robot_gz_control.xacro (robot description, xacro)
@@ -16,5 +16,6 @@
         <wheel_radius>0.165</wheel_radius>
         <!-- Control gains and limits (optional) -->
-        <max_velocity>3.0</max_velocity>
+        <!-- <max_velocity>3.0</max_velocity>  -->
+        <max_velocity>5.0</max_velocity>
         <max_linear_acceleration>1</max_linear_acceleration>
         <min_linear_acceleration>-1</min_linear_acceleration>

File: parc_robot_description/urdf/sensors.xacro (robot description, xacro)
@@ -13,5 +13,5 @@
   <!-- zed2 camera -->
   <xacro:zed2 parent="base_link">
-    <origin xyz="0.36 0 0.11" rpy="0 0 0"/>
+    <origin xyz="0.36 0 0.14" rpy="0 0 0"/>
   </xacro:zed2>
   <!-- gps -->
